Commit message: Added damping and changed mu to match tutorial.

File: urdf/ma1400.xacro (robot description, xacro)
@@ -46,4 +46,22 @@
     </collision>
   </link>
+  <joint
+    name="world2base"
+    type="revolute">
+    <origin
+      xyz="0 0 0"
+      rpy="0 -1.57079632679 0" />
+    <parent
+      link="world" />
+    <child
+      link="base_link" />
+    <axis
+      xyz="0 0 1" />
+    <limit
+      lower="0"
+      upper="0"
+      effort="0"
+      velocity="0" />
+  </joint>
   <link
     name="s_link">
@@ -98,22 +116,4 @@
   </link>
   <joint
-    name="world2base"
-    type="revolute">
-    <origin
-      xyz="0 0 0"
-      rpy="0 -1.57079632679 0" />
-    <parent
-      link="world" />
-    <child
-      link="base_link" />
-    <axis
-      xyz="0 0 1" />
-    <limit
-      lower="0"
-      upper="0"
-      effort="0"
-      velocity="0" />
-  </joint>
-  <joint
     name="base2s"
     type="revolute">
@@ -132,4 +132,6 @@
       effort="0"
       velocity="3.8397" />
+    <dynamics
+      damping="0.7" />
   </joint>
   <link
@@ -190,4 +192,6 @@
       effort="0"
       velocity="3.49066" />
+    <dynamics
+      damping="1.7" />
   </joint>
   <link
@@ -248,4 +252,6 @@
       effort="0"
       velocity="3.83972" />
+    <dynamics
+      damping="1.7" />
   </joint>
   <link
@@ -306,4 +312,6 @@
       effort="14"
       velocity="3.22886" />
+    <dynamics
+      damping="1.7" />
   </joint>
   <link
@@ -364,4 +372,6 @@
       effort="14"
       velocity="2.86234" />
+    <dynamics
+      damping="1.7" />
   </joint>
   <link
@@ -422,5 +432,7 @@
       effort="0.98"
       velocity="10.6465" />
-  </joint>
+  <dynamics
+      damping="0.7" />
+</joint>
   <transmission name="base2s_trans">
     <type>transmission_interface/SimpleTransmission</type>

Commit message: Switched to standard joint naming scheme.

File: urdf/ma1400.xacro (robot description, xacro)
@@ -116,5 +116,5 @@
   </link>
   <joint
-    name="base2s"
+    name="joint_s"
     type="revolute">
     <origin
@@ -176,5 +176,5 @@
   </link>
   <joint
-    name="s2l"
+    name="joint_l"
     type="revolute">
     <origin
@@ -236,5 +236,5 @@
   </link>
   <joint
-    name="l2u"
+    name="joint_u"
     type="revolute">
     <origin
@@ -296,5 +296,5 @@
   </link>
   <joint
-    name="u2r"
+    name="joint_r"
     type="revolute">
     <origin
@@ -356,5 +356,5 @@
   </link>
   <joint
-    name="r2b"
+    name="joint_b"
     type="revolute">
     <origin
@@ -416,5 +416,5 @@
   </link>
   <joint
-    name="b2t"
+    name="joint_t"
     type="revolute">
     <origin
@@ -435,55 +435,55 @@
       damping="0.7" />
 </joint>
-  <transmission name="base2s_trans">
-    <type>transmission_interface/SimpleTransmission</type>
-    <actuator name="$base2s_motor">
-      <mechanicalReduction>1</mechanicalReduction>
-    </actuator>
-    <joint name="base2s">
-      <hardwareInterface>PositionJointInterface</hardwareInterface>
-    </joint>
-  </transmission>
-  <transmission name="s2l_trans">
-    <type>transmission_interface/SimpleTransmission</type>
-    <actuator name="$s2l_motor">
-      <mechanicalReduction>1</mechanicalReduction>
-    </actuator>
-    <joint name="s2l">
-      <hardwareInterface>PositionJointInterface</hardwareInterface>
-    </joint>
-  </transmission>
-  <transmission name="l2u_trans">
-    <type>transmission_interface/SimpleTransmission</type>
-    <actuator name="$l2u_motor">
-      <mechanicalReduction>1</mechanicalReduction>
-    </actuator>
-    <joint name="l2u">
-      <hardwareInterface>PositionJointInterface</hardwareInterface>
-    </joint>
-  </transmission>
-  <transmission name="u2r_trans">
-    <type>transmission_interface/SimpleTransmission</type>
-    <actuator name="$u2r_motor">
-      <mechanicalReduction>1</mechanicalReduction>
-    </actuator>
-    <joint name="u2r">
-      <hardwareInterface>PositionJointInterface</hardwareInterface>
-    </joint>
-  </transmission>
-  <transmission name="r2b_trans">
-    <type>transmission_interface/SimpleTransmission</type>
-    <actuator name="$r2b_motor">
-      <mechanicalReduction>1</mechanicalReduction>
-    </actuator>
-    <joint name="r2b">
-      <hardwareInterface>PositionJointInterface</hardwareInterface>
-    </joint>
-  </transmission>
-  <transmission name="b2t_trans">
-    <type>transmission_interface/SimpleTransmission</type>
-    <actuator name="$b2t_motor">
-      <mechanicalReduction>1</mechanicalReduction>
-    </actuator>
-    <joint name="b2t">
+  <transmission name="s_trans">
+    <type>transmission_interface/SimpleTransmission</type>
+    <actuator name="$s_motor">
+      <mechanicalReduction>1</mechanicalReduction>
+    </actuator>
+    <joint name="joint_s">
+      <hardwareInterface>PositionJointInterface</hardwareInterface>
+    </joint>
+  </transmission>
+  <transmission name="l_trans">
+    <type>transmission_interface/SimpleTransmission</type>
+    <actuator name="$l_motor">
+      <mechanicalReduction>1</mechanicalReduction>
+    </actuator>
+    <joint name="joint_l">
+      <hardwareInterface>PositionJointInterface</hardwareInterface>
+    </joint>
+  </transmission>
+  <transmission name="u_trans">
+    <type>transmission_interface/SimpleTransmission</type>
+    <actuator name="$u_motor">
+      <mechanicalReduction>1</mechanicalReduction>
+    </actuator>
+    <joint name="joint_u">
+      <hardwareInterface>PositionJointInterface</hardwareInterface>
+    </joint>
+  </transmission>
+  <transmission name="r_trans">
+    <type>transmission_interface/SimpleTransmission</type>
+    <actuator name="$r_motor">
+      <mechanicalReduction>1</mechanicalReduction>
+    </actuator>
+    <joint name="joint_r">
+      <hardwareInterface>PositionJointInterface</hardwareInterface>
+    </joint>
+  </transmission>
+  <transmission name="b_trans">
+    <type>transmission_interface/SimpleTransmission</type>
+    <actuator name="$b_motor">
+      <mechanicalReduction>1</mechanicalReduction>
+    </actuator>
+    <joint name="joint_b">
+      <hardwareInterface>PositionJointInterface</hardwareInterface>
+    </joint>
+  </transmission>
+  <transmission name="t_trans">
+    <type>transmission_interface/SimpleTransmission</type>
+    <actuator name="$t_motor">
+      <mechanicalReduction>1</mechanicalReduction>
+    </actuator>
+    <joint name="joint_t">
       <hardwareInterface>PositionJointInterface</hardwareInterface>
     </joint>
