Commit message: Moved stl files to subdirectory.

File: urdf/ma1400.urdf.xacro (robot description, xacro)
@@ -190,5 +190,5 @@
         <origin xyz="0 0 0" rpy="0 0 0" />
         <geometry>
-          <mesh filename="package://ma1400_sim/meshes/${name}_link.stl" />
+          <mesh filename="package://ma1400_sim/meshes/ma1400/${name}_link.stl" />
         </geometry>
         <material name="Cast Carbon Steal">
@@ -199,5 +199,5 @@
         <origin xyz="0 0 0" rpy="0 0 0" />
         <geometry>
-          <mesh filename="package://ma1400_sim/meshes/${name}_link.stl" />
+          <mesh filename="package://ma1400_sim/meshes/ma1400/${name}_link.stl" />
         </geometry>
       </collision>
