Commit message: Adding tailstock and headstock to gazebo.

File: urdf/headstock/headstock.urdf.xacro (robot description, xacro)
@@ -1,4 +1,25 @@
 <?xml version="1.0"?>
 <robot name="headstock" xmlns:xacro="http://www.ros.org/wiki/xacro">
+  <!-- Constants for robot dimensions -->
+  <xacro:property name="M_PI" value="3.1415926535897931"/>
+  <link name="world" />
+    <joint
+    name="joint_base"
+    type="revolute">
+    <origin
+      xyz="2 0.422021 0"
+      rpy="0 ${-M_PI/2} ${-M_PI/2}" />
+    <parent
+      link="world" />
+    <child
+      link="base_link" />
+    <axis
+      xyz="1 0 0" />
+    <limit
+      lower="0"
+      upper="0"
+      effort="0"
+      velocity="0" />
+  </joint>
   <link
     name="base_link">
@@ -41,4 +62,20 @@
     </collision>
   </link>
+  <joint
+    name="joint_revolute"
+    type="revolute">
+    <origin
+      xyz="0.815 0 0.1108"
+      rpy="0 1.5708 0" />
+    <parent
+      link="base_link" />
+    <child
+      link="revolute_link" />
+    <axis
+      xyz="1 0 0" />
+    <limit
+      effort="0"
+      velocity="0" />
+  </joint>
   <link
     name="revolute_link">
@@ -82,16 +119,18 @@
   </link>
   <joint
-    name="joint_revolute"
-    type="revolute">
+    name="joint_prismatic"
+    type="prismatic">
     <origin
-      xyz="0.815 0 0.1108"
-      rpy="0 1.5708 0" />
+      xyz="0.1108 0 0"
+      rpy="3.2816E-38 -3.1907E-15 -1.513E-16" />
     <parent
-      link="base_link" />
+      link="revolute_link" />
     <child
-      link="revolute_link" />
+      link="prismatic_link" />
     <axis
-      xyz="1 0 0" />
+      xyz="0 1 0" />
     <limit
+      lower="0"
+      upper="0"
       effort="0"
       velocity="0" />
@@ -137,21 +176,3 @@
     </collision>
   </link>
-  <joint
-    name="joint_prismatic"
-    type="prismatic">
-    <origin
-      xyz="0.1108 0 0"
-      rpy="3.2816E-38 -3.1907E-15 -1.513E-16" />
-    <parent
-      link="revolute_link" />
-    <child
-      link="prismatic_link" />
-    <axis
-      xyz="0 1 0" />
-    <limit
-      lower="0"
-      upper="0"
-      effort="0"
-      velocity="0" />
-  </joint>
 </robot>

File: urdf/tailstock/tailstock.urdf.xacro (robot description, xacro)
@@ -1,4 +1,25 @@
 <?xml version="1.0"?>
 <robot name="tailstock" xmlns:xacro="http://www.ros.org/wiki/xacro">
+  <!-- Constants for robot dimensions -->
+  <xacro:property name="M_PI" value="3.1415926535897931"/>
+  <link name="world" />
+    <joint
+    name="joint_base"
+    type="revolute">
+    <origin
+      xyz="2 -0.422021 0"
+      rpy="0 ${-M_PI/2} 0" />
+    <parent
+      link="world" />
+    <child
+      link="base_link" />
+    <axis
+      xyz="1 0 0" />
+    <limit
+      lower="0"
+      upper="0"
+      effort="0"
+      velocity="0" />
+  </joint>
   <link
     name="base_link">
@@ -41,4 +62,23 @@
     </collision>
   </link>
+  <joint
+    name="joint_prismatic"
+    type="prismatic">
+    <origin
+      xyz="0.87075 0 -0.2021"
+      rpy="0 1.5708 0" />
+    <parent
+      link="base_link" />
+    <child
+      link="prismatic_link" />
+    <axis
+      xyz="1 0 0" />
+    <!-- Position of link can be controlled here -->
+    <limit
+      lower="0"
+      upper="0"
+      effort="0"
+      velocity="0" />
+  </joint>
   <link
     name="prismatic_link">
@@ -82,18 +122,16 @@
   </link>
   <joint
-    name="joint_prismatic"
-    type="prismatic">
+    name="joint_revolute"
+    type="revolute">
     <origin
-      xyz="0.87075 0 -0.2021"
-      rpy="0 1.5708 0" />
+      xyz="0.095915 0 0"
+      rpy="-4.9284E-29 -4.5181E-15 6.8878E-15" />
     <parent
-      link="base_link" />
+      link="prismatic_link" />
     <child
-      link="prismatic_link" />
+      link="revolute_link" />
     <axis
       xyz="1 0 0" />
     <limit
-      lower="-0.2224"
-      upper="0.2224"
       effort="0"
       velocity="0" />
@@ -139,19 +177,3 @@
     </collision>
   </link>
-  <joint
-    name="joint_revolute"
-    type="revolute">
-    <origin
-      xyz="0.095915 0 0"
-      rpy="-4.9284E-29 -4.5181E-15 6.8878E-15" />
-    <parent
-      link="prismatic_link" />
-    <child
-      link="revolute_link" />
-    <axis
-      xyz="1 0 0" />
-    <limit
-      effort="0"
-      velocity="0" />
-  </joint>
 </robot>

Commit message: Trying to get headstock controller working with ma1400 controller.

File: urdf/headstock/headstock.urdf.xacro (robot description, xacro)
@@ -75,6 +75,8 @@
       xyz="1 0 0" />
     <limit
-      effort="0"
-      velocity="0" />
+      lower="-10000"
+      upper="10000"
+      effort="10"
+      velocity="${2*M_PI}" />
   </joint>
   <link

File: urdf/muffler_00/muffler_00.urdf.xacro (robot description, xacro)
@@ -1,4 +1,30 @@
 <?xml version="1.0"?>
 <robot name="muffler_00" xmlns:xacro="http://www.ros.org/wiki/xacro">
+  <!-- Constants for robot dimensions -->
+  <xacro:property name="M_PI" value="3.1415926535897931"/>
+  <!-- Import all Gazebo-customization elements, including Gazebo colors -->
+  <xacro:include filename="$(find ma1400_sim)/urdf/muffler_00/muffler_00.gazebo.xacro" />
+  <!-- Import trasnmission macro -->
+  <xacro:include filename="$(find ma1400_sim)/urdf/muffler_00/muffler_00.transmission.xacro" />
+  <!-- Add the headstock to the muffler -->
+  <xacro:include filename="$(find ma1400_sim)/urdf/headstock/headstock.urdf.xacro" />
+  <joint
+    name="joint_muffler"
+    type="revolute">
+    <origin
+      xyz="0 0 0"
+      rpy="0 0 0" />
+    <parent
+      link="prismatic_link" />
+    <child
+      link="muffler_link" />
+    <axis
+      xyz="1 0 0" />
+    <limit
+      lower="0"
+      upper="0"
+      effort="0"
+      velocity="0" />
+  </joint>
   <link
     name="muffler_link">
@@ -41,3 +67,4 @@
     </collision>
   </link>
+  <xacro:muffler_00_transmission name="revolute" />
 </robot>

File: urdf/tailstock/tailstock.urdf.xacro (robot description, xacro)
@@ -167,4 +167,5 @@
       </material>
     </visual>
+    <!--
     <collision>
       <origin
@@ -176,4 +177,5 @@
       </geometry>
     </collision>
+    -->
   </link>
 </robot>
