Commit message: Added simplified collision models.

File: urdf/ma1400/ma1400.urdf.xacro (robot description, xacro)
@@ -222,5 +222,5 @@
         <origin xyz="0 0 0" rpy="0 0 0" />
         <geometry>
-          <mesh filename="package://ma1400_sim/meshes/ma1400/${name}_link.stl" />
+          <mesh filename="package://ma1400_sim/meshes/ma1400/${name}_link_collision.stl" />
         </geometry>
       </collision>
